File: hardware/rev_a/buckler.sch (EAGLE design)
At the start: 19 parts, among them J1 ARDUINO_R3_SHIELD_ICSP_NRF528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, J2 DM3AT-SF-PEJM5, U11 SI7021-A20-GM1, U12 SIP32510, U14 MPU-9250, U8 MAX44009, U9 MS5637-02BA03

Commit message: Checkpoint. Done with schematic
Parts:
- added A1: NHD-0216KZWSERIAL, headers:NHD-0216KZWSERIAL
- added C1, C2, C3, C4: 0.1uF, passives:CAPACITOR0402_CAP
- added D1: (no value), passives:DIODE_SCHOTTKYNSR0620P2T5G
- added D2: RED, leds:LED0603
- added D3: GREEN, leds:LED0603
- added D4: BLUE, leds:LED0603
- added D5: YELLOW, leds:LED0603
- added J3: DB25_5747846, headers:DB25_5747846
- added J4, J5, J6, J7, J8, J9: 4P-2.0, headers:GROVE-CONNECTOR-DIP(4P-2.0)
- added R10, R11, R2, R3, R4: 10k, passives:RESISTOR0402_RES
- added R5, R6, R7, R8: 1k, passives:RESISTOR0402_RES
- added S1, S3, S7: PTS645SM43SMTR92, switches:PTS645SM43SMTR92
- added S2: B3U-1000P, switches:B3U-1000P
- added S25, S4: TE_SSA12/SPDT, switches:TE_SSA12/SPDT
- added TP1, TP2, TP27, TP28, TP3, TP4, TP5: TEST_POINT_0.040IN, headers:TEST_POINT_0.040IN
- added U1: ADXL327, chips:ADXL327
- J1: value ARDUINO_R3_SHIELD_ICSP_NRF52840DK -> NRF52840DK_SHIELD; device headers:ARDUINO_R3_SHIELD_ICSP_NRF52840DK -> headers:NRF52840DK_SHIELD
Connections:
- removed net !IMU_INT: R1.1, U14.INT
- removed net !LT_INT: R9.1, U8.!INT
- removed net N$34: U9.SCL
- removed net N$41: U9.SDA
- removed net N$50: U11.SCL
- removed net N$51: U8.SDA
- removed net N$52: U8.SCL
- new net !BUTTON_0: J1.P1.12, R10.1, S1.P$1
- new net !BUTTON_1: J1.P1.13, R11.1, S3.P$1
- new net !IMU_INTERRUPT: J1.P1.01, R1.1, TP5.TESTPOINT, U14.INT
- new net !LCD_CS: A1.!CS, J1.P1.03
- new net !LED_0: D2.CATHODE, J1.P1.06
- new net !LED_1: D3.CATHODE, J1.P1.07
- new net !LED_2: D4.CATHODE, J1.P1.10
- new net !LED_3: D5.CATHODE, J1.P1.11
- new net !LIGHT_INTERRUPT: J1.P1.02, R9.1, TP4.TESTPOINT, U8.!INT
- new net ANALOG_ACCEL_X: C4.1, J1.P0.29/AIN5, TP28.TESTPOINT, U1.XOUT
- new net ANALOG_ACCEL_Y: C3.1, J1.P0.30/AIN6, TP27.TESTPOINT, U1.YOUT
- new net ANALOG_ACCEL_Z: C2.1, J1.P0.31/AIN7, TP1.TESTPOINT, U1.ZOUT
- new net EXTERN_RX: J1.P0.25, J3.1, J5.2
- new net EXTERN_TX: J1.P0.24, J3.2, J5.1
- new net GROVE_A0: J1.P0.02/AIN0, J6.1
- new net GROVE_A1: J1.P0.03/AIN1, J6.2
- new net GROVE_A2: J1.P0.28/AIN4, J7.1
- new net GROVE_D0: J1.P0.04/AIN2, J8.1
- new net GROVE_D1: J1.P1.08, J8.2
- new net GROVE_D2: J1.P1.09, J9.1
- new net LCD_MISO: A1.MISO, J1.P0.14
- new net LCD_MOSI: A1.MOSI, J1.P0.16
- new net LCD_SCLK: A1.SCLK, J1.P0.12
- new net N$2: D1.ANODE, J3.8, J3.9
- new net N$25: D2.ANODE, R5.2
- new net N$3: D3.ANODE, R6.2
- new net N$4: D4.ANODE, R7.2
- new net N$5: D5.ANODE, R8.2
- new net N$7: S2.P$1, U1.ST
- new net SWITCH_0: J1.P1.14, S25.IN
- new net SWITCH_1: J1.P1.15, S4.IN
- net !SD_CS: now also J1.P1.04
- net !SD_DETECT: now also J1.P1.05
- net +3V3: now also A1.VCC, C1.1, J4.3, J5.3, J6.3, J7.3, J8.3, J9.3, R10.2, R11.2, R2.2, R3.2, R4.2, R5.1, R6.1, R7.1, R8.1, S2.P$2, S25.B, S4.B, U1.VCC
- net +5V: now also D1.CATHODE
- net GND: now also A1.GND, C1.2, C2.2, C3.2, C4.2, J3.16, J3.20, J3.21, J3.24, J3.25, J3.6, J4.4, J5.4, J6.4, J7.4, J8.4, J9.4, S1.P$2, S25.A, S3.P$2, S4.A, S7.P$2, U1.GND
- net N$1: now also J1.P0.18/!RESET, R2.1, S7.P$1; no longer U11.SDA
- net SD_MISO: now also J1.P0.13
- net SD_MOSI: now also J1.P0.15
- net SD_SCLK: now also J1.P0.11
- net SENSORS_SCL: now also J1.P0.27, J4.1, R3.1, TP3.TESTPOINT, U11.SCL, U8.SCL, U9.SCL
- net SENSORS_SDA: now also J1.P0.26, J4.2, R4.1, TP2.TESTPOINT, U11.SDA, U8.SDA, U9.SDA
Other:
- note added: "2x16 LCD Screen"
- note added: "3-Axis Accelerometer/Gyro/Magnetometer"
- note added: "Analog Accelerometer"
- note added: "DB-25 Header for Kobuki"
- note added: "Grove Headers"
- note added: "I2C Address: 0x40"
- note added: "I2C Address: 0x4A"
- note added: "I2C Address: 0x76"
- note added: "I2C Bus"
- note added: "LEDs (Various Colors)"
- note added: "Push Buttons (Momentary)"
- note added: "Self Test Button"
- note added: "Switches"
- note added: "UART shared with Kobuki"
- note added: "nRF52840DK Interface"
- note removed: "Accelerometer/Gyro/Magnetometer"
- moved on the sheet: C18, C19, C20, C25, C26, J2, R1, R12, R13, R14, R16, R17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

Commit message: Checkpoint. 50 airwares remaining!
Parts:
- removed TP1, TP2, TP27, TP28, TP3: TEST_POINT_0.040IN, headers:TEST_POINT_0.040IN
- added TP10, TP11, TP12, TP13, TP14, TP15, TP16, TP17, TP18, TP19, TP20, TP21, TP22, TP23, TP24, TP25, TP26, TP29, TP30, TP31, TP32, TP33, TP34, TP35, TP36, TP37, TP38, TP39, TP40, TP41, TP42, TP43, TP44, TP6, TP7, TP8, TP9: TEST_POINT_0.040IN, headers:TEST_POINT_0.040IN
Connections:
- net !BUTTON_0: now also TP36.TESTPOINT
- net !BUTTON_1: now also TP37.TESTPOINT
- net !IMU_INTERRUPT: now also TP6.TESTPOINT; no longer TP5.TESTPOINT
- net !LCD_CS: now also TP8.TESTPOINT
- net !LED_0: now also TP11.TESTPOINT
- net !LED_1: now also TP12.TESTPOINT
- net !LED_2: now also TP13.TESTPOINT
- net !LED_3: now also TP35.TESTPOINT
- net !LIGHT_INTERRUPT: now also TP7.TESTPOINT; no longer TP4.TESTPOINT
- net !SD_CS: now also TP9.TESTPOINT
- net !SD_DETECT: now also TP10.TESTPOINT
- net +3V3: now also TP4.TESTPOINT, TP40.TESTPOINT, TP5.TESTPOINT
- net +5V: now also TP41.TESTPOINT
- net ANALOG_ACCEL_X: now also TP17.TESTPOINT; no longer TP28.TESTPOINT
- net ANALOG_ACCEL_Y: now also TP18.TESTPOINT; no longer TP27.TESTPOINT
- net ANALOG_ACCEL_Z: now also TP19.TESTPOINT; no longer TP1.TESTPOINT
- net EXTERN_RX: now also TP32.TESTPOINT
- net EXTERN_TX: now also TP33.TESTPOINT
- net GND: now also TP42.TESTPOINT, TP43.TESTPOINT, TP44.TESTPOINT
- net GROVE_A0: now also TP14.TESTPOINT
- net GROVE_A1: now also TP15.TESTPOINT
- net GROVE_A2: now also TP16.TESTPOINT
- net GROVE_D0: now also TP34.TESTPOINT
- net GROVE_D1: now also TP29.TESTPOINT
- net GROVE_D2: now also TP26.TESTPOINT
- net LCD_MISO: now also TP22.TESTPOINT
- net LCD_MOSI: now also TP20.TESTPOINT
- net LCD_SCLK: now also TP24.TESTPOINT
- net SD_MISO: now also TP23.TESTPOINT
- net SD_MOSI: now also TP21.TESTPOINT
- net SD_SCLK: now also TP25.TESTPOINT
- net SENSORS_SCL: now also TP30.TESTPOINT; no longer TP3.TESTPOINT
- net SENSORS_SDA: now also TP31.TESTPOINT; no longer TP2.TESTPOINT
- net SWITCH_0: now also TP38.TESTPOINT
- net SWITCH_1: now also TP39.TESTPOINT
Other:
- moved on the sheet: C2, C3, C4

Commit message: Routing complete!!
Parts:
- added C13: 10nF, passives:CAPACITOR0402_CAP
- added C5: 100nF, passives:CAPACITOR0402_CAP
Connections:
- removed net !LED_3: D5.CATHODE, J1.P1.11, TP35.TESTPOINT
- net !LED_1: now also D5.CATHODE; no longer D3.CATHODE
- net +3V3: now also C13.1, C5.1
- net GND: now also C13.2, C5.2, D3.CATHODE
- net N$3: now also R8.2; no longer R6.2
- net N$5: now also R6.2; no longer R8.2
- net SD_ENABLE: now also J1.P1.11, TP35.TESTPOINT
Other:
- moved on the sheet: D2, D3, D4, D5, R5, R6, R7, R8

Commit message: Renumber script, plus some manual tweaks
Parts:
- removed C13: 10nF, passives:CAPACITOR0402_CAP
- removed C18: 100nF, passives:CAPACITOR0402_CAP
- removed C19, C20: 0.1uF, passives:CAPACITOR0402_CAP
- removed C25: 1uF, passives:CAPACITOR0402_CAP
- removed R17: 100k, passives:RESISTOR0402_RES
- removed S7: PTS645SM43SMTR92, switches:PTS645SM43SMTR92
- removed TP40, TP41, TP42, TP43, TP44: TEST_POINT_0.040IN, headers:TEST_POINT_0.040IN
- added C10, C6, C7, C8, C9: 100nF, passives:CAPACITOR0402_CAP
- added R15: 100k, passives:RESISTOR0402_RES
- added S6: TE_SSA12/SPDT, switches:TE_SSA12/SPDT
- added TP1, TP2, TP27, TP28, TP3: TEST_POINT_0.040IN, headers:TEST_POINT_0.040IN
- C1: value 0.1uF -> 10nF; DESCRIPTION (none) -> CAP CER 10000PF 50V X7R 0402; DIGIKEY 490-6328-1-ND -> 490-7763-1-ND; MANUFACTURER (none) -> Murata; MPN GRM155R71C104KA88J -> GRM155R71H103JA88D
- C2: value 0.1uF -> 100nF; DESCRIPTION (none) -> CAP CER 0.1UF 10V X7R 0402; DIGIKEY 490-6328-1-ND -> 490-10777-1-ND; MANUFACTURER (none) -> Murata; MPN GRM155R71C104KA88J -> GRM155R71A104JA01D
- C3: value 0.1uF -> 100nF; DIGIKEY 490-6328-1-ND -> 490-7195-1-ND; MPN GRM155R71C104KA88J -> GRM155R70G105KA12D
- C4: value 0.1uF -> 100nF
- C5: DESCRIPTION CAP CER 0.1UF 10V X7R 0402 -> (none); DIGIKEY 490-10777-1-ND -> 490-6328-1-ND; MANUFACTURER Murata -> (none); MPN GRM155R71A104JA01D -> GRM155R71C104KA88J
- D3: value GREEN -> YELLOW; DIGIKEY 160-1435-1-ND -> 160-1437-1-ND
- D5: value YELLOW -> GREEN; DIGIKEY 160-1437-1-ND -> 160-1435-1-ND
- J1: value NRF52840DK_SHIELD -> DB25_5747846; device headers:NRF52840DK_SHIELD -> headers:DB25_5747846
- J3: value DB25_5747846 -> 4P-2.0; device headers:DB25_5747846 -> headers:GROVE-CONNECTOR-DIP(4P-2.0)
- J9: value 4P-2.0 -> NRF52840DK_SHIELD; device headers:GROVE-CONNECTOR-DIP(4P-2.0) -> headers:NRF52840DK_SHIELD
- R1, R2, R3, R4: value 10k -> 1k; DESCRIPTION (none) -> RES SMD 1K OHM 1% 1/16W 0402; DIGIKEY 311-10KJRCT-ND -> RMCF0402FT1K00CT-ND; MANUFACTURER (none) -> Stackpole Electronics; MPN RC0402JR-0710KL -> RMCF0402FT1K00
- R12, R13, R14: DESCRIPTION RES SMD 10K OHM 1% 1/16W 0402 -> (none); DIGIKEY RMCF0402FT10K0CT-ND -> 311-10KJRCT-ND; MANUFACTURER Stackpole Electronics -> (none); MPN RMCF0402FT10K0 -> RC0402JR-0710KL
- R5, R6: value 1k -> 10k; DESCRIPTION RES SMD 1K OHM 1% 1/16W 0402 -> (none); DIGIKEY RMCF0402FT1K00CT-ND -> 311-10KJRCT-ND; MANUFACTURER Stackpole Electronics -> (none); MPN RMCF0402FT1K00 -> RC0402JR-0710KL
- R7, R8: value 1k -> 10k; DESCRIPTION RES SMD 1K OHM 1% 1/16W 0402 -> RES SMD 10K OHM 1% 1/16W 0402; DIGIKEY RMCF0402FT1K00CT-ND -> RMCF0402FT10K0CT-ND; MPN RMCF0402FT1K00 -> RMCF0402FT10K0
- R9: DESCRIPTION (none) -> RES SMD 10K OHM 1% 1/16W 0402; DIGIKEY 311-10KJRCT-ND -> RMCF0402FT10K0CT-ND; MANUFACTURER (none) -> Stackpole Electronics; MPN RC0402JR-0710KL -> RMCF0402FT10K0
- S1: value PTS645SM43SMTR92 -> B3U-1000P; device switches:PTS645SM43SMTR92 -> switches:B3U-1000P; MPN (none) -> B3U-1000P
- S2: value B3U-1000P -> PTS645SM43SMTR92; device switches:B3U-1000P -> switches:PTS645SM43SMTR92; MPN B3U-1000P -> (none)
- S4: value TE_SSA12/SPDT -> PTS645SM43SMTR92; device switches:TE_SSA12/SPDT -> switches:PTS645SM43SMTR92
- renumbered C26 to C11, S25 to S5, U11 to U5, U12 to U6, U14 to U3, U8 to U2, U9 to U4
Connections:
- net !BUTTON_0: now also J9.P1.12, R13.1, S3.P$1, TP29.TESTPOINT; no longer J1.P1.12, R10.1, S1.P$1, TP36.TESTPOINT
- net !BUTTON_1: now also J9.P1.13, R14.1, S4.P$1, TP30.TESTPOINT; no longer J1.P1.13, R11.1, S3.P$1, TP37.TESTPOINT
- net !IMU_INTERRUPT: now also J9.P1.01, R6.1, TP1.TESTPOINT; no longer J1.P1.01, R1.1, TP6.TESTPOINT
- net !LCD_CS: now also J9.P1.03, TP3.TESTPOINT; no longer J1.P1.03, TP8.TESTPOINT
- net !LED_0: now also J9.P1.06, TP6.TESTPOINT; no longer J1.P1.06, TP11.TESTPOINT
- net !LED_1: now also D3.CATHODE, J9.P1.07, TP7.TESTPOINT; no longer D5.CATHODE, J1.P1.07, TP12.TESTPOINT
- net !LED_2: now also J9.P1.10, TP8.TESTPOINT; no longer J1.P1.10, TP13.TESTPOINT
- net !LIGHT_INTERRUPT: now also J9.P1.02, R5.1, TP2.TESTPOINT; no longer J1.P1.02, R9.1, TP7.TESTPOINT
- net !SD_CS: now also J9.P1.04, R8.1, TP4.TESTPOINT; no longer J1.P1.04, R13.1, TP9.TESTPOINT
- net !SD_DETECT: now also J9.P1.05, R15.1, TP5.TESTPOINT; no longer J1.P1.05, R16.1, TP10.TESTPOINT
- net +3V3: now also C10.1, C3.1, C4.1, C6.1, J3.3, J9.3.3V, R1.1, R12.2, R13.2, R14.2, R16.2, R2.1, R3.1, R4.1, R5.2, R6.2, S1.P$2, S6.B, TP33.TESTPOINT, TP34.TESTPOINT, TP35.TESTPOINT; no longer C13.1, C19.1, C20.1, C25.1, J1.3.3V, J9.3, R1.2, R17.2, R2.2, R3.2, R4.2, R5.1, R6.1, R7.1, R8.1, R9.2, S2.P$2, S4.B, TP4.TESTPOINT, TP40.TESTPOINT, TP5.TESTPOINT
- net +5V: now also J9.5V, TP36.TESTPOINT; no longer J1.5V, TP41.TESTPOINT
- net ANALOG_ACCEL_X: now also C9.1, J9.P0.29/AIN5, TP12.TESTPOINT; no longer C4.1, J1.P0.29/AIN5, TP17.TESTPOINT
- net ANALOG_ACCEL_Y: now also C8.1, J9.P0.30/AIN6, TP13.TESTPOINT; no longer C3.1, J1.P0.30/AIN6, TP18.TESTPOINT
- net ANALOG_ACCEL_Z: now also C7.1, J9.P0.31/AIN7, TP14.TESTPOINT; no longer C2.1, J1.P0.31/AIN7, TP19.TESTPOINT
- net EXTERN_RX: now also J1.1, J4.2, J9.P0.25, TP25.TESTPOINT; no longer J1.P0.25, J3.1, J5.2, TP32.TESTPOINT
- net EXTERN_TX: now also J1.2, J4.1, J9.P0.24, TP26.TESTPOINT; no longer J1.P0.24, J3.2, J5.1, TP33.TESTPOINT
- net GND: now also C10.2, C6.2, C7.2, C8.2, C9.2, D5.CATHODE, J1.16, J1.20, J1.21, J1.24, J1.25, J1.6, J3.4, J9.GND, S2.P$2, S4.P$2, S6.A, TP37.TESTPOINT, TP38.TESTPOINT, TP39.TESTPOINT; no longer C13.2, C18.2, C19.2, C20.2, C25.2, D3.CATHODE, J1.GND, J3.16, J3.20, J3.21, J3.24, J3.25, J3.6, J9.4, S1.P$2, S4.A, S7.P$2, TP42.TESTPOINT, TP43.TESTPOINT, TP44.TESTPOINT
- net GROVE_A0: now also J5.1, J9.P0.02/AIN0, TP9.TESTPOINT; no longer J1.P0.02/AIN0, J6.1, TP14.TESTPOINT
- net GROVE_A1: now also J5.2, J9.P0.03/AIN1, TP10.TESTPOINT; no longer J1.P0.03/AIN1, J6.2, TP15.TESTPOINT
- net GROVE_A2: now also J6.1, J9.P0.28/AIN4, TP11.TESTPOINT; no longer J1.P0.28/AIN4, J7.1, TP16.TESTPOINT
- net GROVE_D0: now also J7.1, J9.P0.04/AIN2, TP27.TESTPOINT; no longer J1.P0.04/AIN2, J8.1, TP34.TESTPOINT
- net GROVE_D1: now also J7.2, J9.P1.08, TP22.TESTPOINT; no longer J1.P1.08, J8.2, TP29.TESTPOINT
- net GROVE_D2: now also J8.1, J9.P1.09, TP21.TESTPOINT; no longer J1.P1.09, J9.1, TP26.TESTPOINT
- net LCD_MISO: now also J9.P0.14, TP17.TESTPOINT; no longer J1.P0.14, TP22.TESTPOINT
- net LCD_MOSI: now also J9.P0.16, TP15.TESTPOINT; no longer J1.P0.16, TP20.TESTPOINT
- net LCD_SCLK: now also J9.P0.12, TP19.TESTPOINT; no longer J1.P0.12, TP24.TESTPOINT
- net N$1: now also J9.P0.18/!RESET, R10.1, S2.P$1; no longer J1.P0.18/!RESET, R2.1, S7.P$1
- net N$18: now also R15.2, R7.2, R8.2, R9.2; no longer R12.2, R13.2, R14.2, R16.2
- net N$19: now also C2.1; no longer C18.1
- net N$2: now also J1.8, J1.9; no longer J3.8, J3.9
- net N$25: now also R1.2; no longer R5.2
- net N$3: now also D5.ANODE, R4.2; no longer D3.ANODE, R8.2
- net N$4: now also R3.2; no longer R7.2
- net N$5: now also D3.ANODE, R2.2; no longer D5.ANODE, R6.2
- net N$7: now also S1.P$1; no longer S2.P$1
- net SD_ENABLE: now also J9.P1.11, R16.1, TP28.TESTPOINT; no longer J1.P1.11, R17.1, TP35.TESTPOINT
- net SD_MISO: now also J9.P0.13, R9.1, TP18.TESTPOINT; no longer J1.P0.13, R14.1, TP23.TESTPOINT
- net SD_MOSI: now also J9.P0.15, R7.1, TP16.TESTPOINT; no longer J1.P0.15, R12.1, TP21.TESTPOINT
- net SD_SCLK: now also J9.P0.11, TP20.TESTPOINT; no longer J1.P0.11, TP25.TESTPOINT
- net SENSORS_SCL: now also J3.1, J9.P0.27, R11.1, TP23.TESTPOINT; no longer J1.P0.27, J4.1, R3.1, TP30.TESTPOINT
- net SENSORS_SDA: now also J3.2, J9.P0.26, R12.1, TP24.TESTPOINT; no longer J1.P0.26, J4.2, R4.1, TP31.TESTPOINT
- net SWITCH_0: now also J9.P1.14, TP31.TESTPOINT; no longer J1.P1.14, TP38.TESTPOINT
- net SWITCH_1: now also J9.P1.15, S6.IN, TP32.TESTPOINT; no longer J1.P1.15, S4.IN, TP39.TESTPOINT

Commit message: Checkpoint, adding part numbers
Parts:
- added TP40, TP41, TP42: TEST_POINT_0.040IN, headers:TEST_POINT_0.040IN
- C1: DESCRIPTION CAP CER 10000PF 50V X7R 0402 -> CAP CER 10000PF 25V X7R 0402; DIGIKEY 490-7763-1-ND -> 399-1279-1-ND; MANUFACTURER Murata -> KEMET; MPN GRM155R71H103JA88D -> C0402C103J3RACTU
- C10, C2: DESCRIPTION CAP CER 0.1UF 10V X7R 0402 -> CAP CER 0.1UF 16V X7R 0402; DIGIKEY 490-10777-1-ND -> 490-4759-1-ND; MPN GRM155R71A104JA01D -> GCM155R71C104KA55D
- C11: DESCRIPTION CAP CER 4.7UF 6.3V X5R 0402 -> CAP CER 4.7UF 10V X5R 0402; DIGIKEY 445-5947-1-ND -> 1276-1480-1-ND; MANUFACTURER TDK -> Samsung Electro-Mechanics; MPN C1005X5R0J475K050BC -> CL05A475KP5NRNC
- C3: DESCRIPTION (none) -> CAP CER 0.1UF 16V X7R 0402; DIGIKEY 490-7195-1-ND -> 490-4759-1-ND; MANUFACTURER (none) -> Murata; MPN GRM155R70G105KA12D -> GCM155R71C104KA55D
- C4, C5, C6, C7, C8, C9: DESCRIPTION (none) -> CAP CER 0.1UF 16V X7R 0402; DIGIKEY 490-6328-1-ND -> 490-4759-1-ND; MANUFACTURER (none) -> Murata; MPN GRM155R71C104KA88J -> GCM155R71C104KA55D
- D1: device passives:DIODE_SCHOTTKYNSR0620P2T5G -> passives:DIODE_SCHOTTKYSOD323; DESCRIPTION (none) -> DIODE SCHOTTKY 30V 500MA SOD323; DIGIKEY (none) -> B0530WS-FDICT-ND; MANUFACTURER (none) -> Diodes Incorporated; MPN (none) -> B0530WS-7-F
- D2: DESCRIPTION (none) -> LED RED CLEAR CHIP SMD; MANUFACTURER (none) -> Lite-On Inc.; MPN (none) -> LTST-C190KRKT
- D3: DESCRIPTION (none) -> LED YELLOW CLEAR CHIP SMD; MANUFACTURER (none) -> Lite-On Inc.; MPN (none) -> LTST-C190KSKT
- D4: DESCRIPTION (none) -> LED BLUE CLEAR SMD; MANUFACTURER (none) -> Lite-On Inc.; MPN (none) -> LTST-C194TBKT
- D5: DESCRIPTION (none) -> LED GREEN CLEAR CHIP SMD; MANUFACTURER (none) -> Lite-On Inc.; MPN (none) -> LTST-C190KGKT
- J1: DESCRIPTION (none) -> CONN D-SUB RCPT 25POS R/A SOLDER; MANUFACTURER (none) -> TE Connectivity AMP Connectors; MPN (none) -> 5747846-4
- J3, J4, J5, J6, J7, J8: DESCRIPTION (none) -> Grove - Universal 4 pin connector; MANUFACTURER (none) -> Seeed Studio; MOUSER (none) -> 713-110990030; MPN (none) -> 110990030
- R5, R6: DESCRIPTION (none) -> RES SMD 10K OHM 1% 1/16W 0402; DIGIKEY 311-10KJRCT-ND -> 1276-3431-1-ND; MANUFACTURER (none) -> Samsung Electro-Mechanics; MPN RC0402JR-0710KL -> RC1005F103CS
- R7, R8: DIGIKEY RMCF0402FT10K0CT-ND -> 1276-3431-1-ND; MANUFACTURER Stackpole Electronics -> Samsung Electro-Mechanics; MPN RMCF0402FT10K0 -> RC1005F103CS
Connections:
- net GND: now also TP40.TESTPOINT, TP41.TESTPOINT, TP42.TESTPOINT

Commit message: Finished add part numbers for everything
Parts:
- A1: DIGIKEY1 (none) -> NHD-0216KZW-AG5-ND; DIGIKEY2 (none) -> 952-3305-ND
- J9: DESCRIPTION (none) -> Headers for nRF52840DK. There are 6 separate headers to be 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; DIGIKEY1 (none) -> S1011EC-10-ND; DIGIKEY2 (none) -> S1011EC-08-ND; DIGIKEY3 (none) -> S1011EC-08-ND; DIGIKEY4 (none) -> S1011EC-08-ND; DIGIKEY5 (none) -> S1011EC-06-ND; DIGIKEY6 (none) -> S2011EC-09-ND
- R10, R11, R12, R13, R14: DESCRIPTION (none) -> RES SMD 10K OHM 1% 1/16W 0402; DIGIKEY 311-10KJRCT-ND -> 1276-3431-1-ND; MANUFACTURER (none) -> Samsung Electro-Mechanics; MPN RC0402JR-0710KL -> RC1005F103CS
- R15, R16: DESCRIPTION RES SMD 100K OHM 1% 1/16W 0402 -> RES SMD 100K OHM 1% 1/5W 0402; DIGIKEY 1276-3432-1-ND -> 541-100KYCT-ND; MANUFACTURER Samsung -> Vishay Dale; MPN RC1005F104CS -> CRCW0402100KFKEDHP
- R9: DIGIKEY RMCF0402FT10K0CT-ND -> 1276-3431-1-ND; MANUFACTURER Stackpole Electronics -> Samsung Electro-Mechanics; MPN RMCF0402FT10K0 -> RC1005F103CS
- S1: DESCRIPTION (none) -> SWITCH TACTILE SPST-NO 0.05A 12V
- S2, S3, S4: DESCRIPTION (none) -> SWITCH TACTILE SPST-NO 0.05A 12V; MANUFACTURER (none) -> C&K; MPN (none) -> PTS645SM43SMTR92 LFS
- S5, S6: DESCRIPTION (none) -> SWITCH SLIDE SPDT 100MA 30V; MANUFACTURER (none) -> TE Connectivity ALCOSWITCH Switches; MPN (none) -> SSA12
- U1: DESCRIPTION (none) -> ACCELEROMETER 2G ANALOG 16LFCSP; MANUFACTURER (none) -> Analog Devices Inc.; MPN (none) -> ADXL327BCPZ
- U2: DESCRIPTION (none) -> SENSOR AMBIENT LIGHT 6UTDFN; MANUFACTURER (none) -> Maxim Integrated
- U3: DESCRIPTION (none) -> IMU ACCEL/GYRO/MAG I2C/SPI 24QFN; MANUFACTURER (none) -> TDK InvenSense; MPN (none) -> MPU-9250
- U4: DESCRIPTION (none) -> SENSOR 17.4PSIA I2C 24B 4-QFN
- U5: DESCRIPTION (none) -> SENS HUMI/TEMP 3.6V I2C 3% 6DFN; MANUFACTURER (none) -> Silicon Labs
- U6: DESCRIPTION (none) -> IC LOAD SWITCH SOT23-6

Commit message: Silkscreen complete
Parts:
- added TP43, TP44: TEST_POINT_0.078IN, headers:TEST_POINT_0.078IN
Connections:
- net GND: now also TP43.TESTPOINT, TP44.TESTPOINT
Other:
- note added: "Clippable Ground Pins"
Changed lines of the file:
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@@
 <attribute name="MPN" value="B0530WS-7-F"/>
 </part>
+<part name="TP43" library="headers" deviceset="TEST_POINT_0.078IN" device="">
+<attribute name="DESCRIPTION" value="TERM TURRET SINGLE L=4.75MM TIN"/>
+<attribute name="DIGIKEY" value="36-1520-2-ND"/>
+<attribute name="MANUFACTURER" value="Keystone Electronics"/>
+<attribute name="MPN" value="1520-2"/>
+</part>
+<part name="TP44" library="headers" deviceset="TEST_POINT_0.078IN" device="">
+<attribute name="DESCRIPTION" value="TERM TURRET SINGLE L=4.75MM TIN"/>
+<attribute name="DIGIKEY" value="36-1520-2-ND"/>
+<attribute name="MANUFACTURER" value="Keystone Electronics"/>
+<attribute name="MPN" value="1520-2"/>
+</part>
+<part name="GND27" library="regulators" deviceset="GND" device=""/>
 </parts>
 <sheets>
@@
 <text x="231.14" y="132.08" size="2.032" layer="98">UART shared
 with Kobuki</text>
+<text x="111.76" y="66.04" size="2.54" layer="98">Clippable
+Ground Pins</text>
 </plain>
 <instances>
@@
 <attribute name="MPN" x="45.72" y="55.88" size="1.778" layer="96" rot="R90" display="off"/>
 </instance>
+<instance part="TP43" gate="G$1" x="116.84" y="63.5">
+<attribute name="DESCRIPTION" x="116.84" y="63.5" size="1.778" layer="96" display="off"/>
+<attribute name="DIGIKEY" x="116.84" y="63.5" size="1.778" layer="96" display="off"/>
+<attribute name="MANUFACTURER" x="116.84" y="63.5" size="1.778" layer="96" display="off"/>
+<attribute name="MPN" x="116.84" y="63.5" size="1.778" layer="96" display="off"/>
+</instance>
+<instance part="TP44" gate="G$1" x="116.84" y="60.96">
+<attribute name="DESCRIPTION" x="116.84" y="60.96" size="1.778" layer="96" display="off"/>
+<attribute name="DIGIKEY" x="116.84" y="60.96" size="1.778" layer="96" display="off"/>
+<attribute name="MANUFACTURER" x="116.84" y="60.96" size="1.778" layer="96" display="off"/>
+<attribute name="MPN" x="116.84" y="60.96" size="1.778" layer="96" display="off"/>
+</instance>
+<instance part="GND27" gate="G1" x="121.92" y="55.88"/>
 </instances>
 <busses>
@@
 <wire x1="213.36" y1="93.98" x2="213.36" y2="91.44" width="0.1524" layer="91"/>
 </segment>
+<segment>
+<pinref part="TP43" gate="G$1" pin="TESTPOINT"/>
+<wire x1="119.38" y1="63.5" x2="121.92" y2="63.5" width="0.1524" layer="91"/>
+<wire x1="121.92" y1="63.5" x2="121.92" y2="60.96" width="0.1524" layer="91"/>
+<pinref part="TP44" gate="G$1" pin="TESTPOINT"/>
+<wire x1="121.92" y1="60.96" x2="119.38" y2="60.96" width="0.1524" layer="91"/>
+<pinref part="GND27" gate="G1" pin="GND"/>
+<wire x1="121.92" y1="58.42" x2="121.92" y2="60.96" width="0.1524" layer="91"/>
+<junction x="121.92" y="60.96"/>
+</segment>
 </net>

Commit message: Finished with schematic and layout for rev A
Parts:
- C10: value 100nF -> 1uF; DESCRIPTION CAP CER 0.1UF 16V X7R 0402 -> CAP CER 1UF 10V X6S 0402; DIGIKEY 490-4759-1-ND -> 1276-6805-1-ND; MANUFACTURER Murata -> Samsung Electro-Mechanics; MPN GCM155R71C104KA55D -> CL05X105KP5NNNC
Connections:
- net +3V3: now also C9.1; no longer C6.1
- net ANALOG_ACCEL_X: now also C8.1; no longer C9.1
- net ANALOG_ACCEL_Y: now also C7.1; no longer C8.1
- net ANALOG_ACCEL_Z: now also C6.1; no longer C7.1
Other:
- note added: "Power Indicator"
- moved on the sheet: C10, C3, C4, C5, C6, C7, C8, C9
