File: hardware/rev_b/buckler.brd (EAGLE design)
At the start: 63.5 x 114.3 mm, 91 parts, among them J1 DB25_5747846, J2 DM3AT-SF-PEJM5, J3 4P-2.0, J4 4P-2.0, J5 4P-2.0, J6 NRF52832DK_SHIELD, J7 4P-2.0, U1 ADXL327, U2 MAX44009, U3 MPU-9250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

Commit message: Routing complete
Parts:
- moved J4 38.1 mm to (55.9, 10.2)
- moved J5 38.1 mm to (17.8, 10.2)
- moved J3 12.7 mm to (43.2, 10.2)
- moved J7 12.7 mm to (30.5, 10.2)
- moved R8 9.58 mm to (20.3, 87.2), turned to 270 degrees
- moved TP5 6.10 mm to (27.1, 100.7)
- moved R4 5.57 mm to (24.1, 103.8)
- moved TP10 2.54 mm to (1.91, 57.1)
- moved TP9 2.54 mm to (1.91, 54.6)
- moved A1 0.63 mm to (50.2, 105.4)
- moved R10 0.63 mm to (24.1, 106.0)
- moved R12 0.63 mm to (53.3, 92.1)
Connections:
- net N$1 renamed !RESET
- net N$2 renamed 5V_IN
- removed net EXTERN_RX: J1.1, J4.2
- net GROVE_A0: now also J6.P0.04; no longer J6.P0.03
- net GROVE_A1: now also J6.P0.03; no longer J6.P0.04
- net UART_RX: now also J1.1, J4.2
Routing:
- net SENSORS_SCL: track 5.71 -> 162.3 mm, vias 0 -> 6
- net SENSORS_SDA: track 5.71 -> 158.6 mm, vias 0 -> 4
- net !RESET: track 13.7 -> 153.3 mm, vias 0 -> 3
- net SWITCH_0: track 5.71 -> 120.0 mm, vias 0 -> 5
- net GROVE_D0: track 5.71 -> 102.6 mm, vias 0 -> 6
- net !LED_0: track 5.71 -> 96.5 mm, vias 0 -> 4
- net SD_MISO: track 5.71 -> 94.7 mm
- net !LED_1: track 5.71 -> 93.3 mm, vias 0 -> 4
- net !LED_2: track 5.71 -> 90.0 mm, vias 0 -> 4
- net SD_MOSI: track 5.71 -> 88.9 mm, vias 0 -> 2
- net SD_SCLK: track 5.71 -> 84.4 mm
- net 5V_IN: track 0.00 -> 78.0 mm, vias 0 -> 2
- net !SD_CS: track 5.71 -> 81.5 mm
- net GND: track 15.9 -> 83.4 mm, vias 0 -> 19
- net GROVE_A1: track 5.71 -> 61.9 mm, vias 0 -> 2
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Other:
- board text added: "!BUTTON_0"
- board text added: "!IMU_INT"
- board text added: "!LCD_CS"
- board text added: "!LED_0"
- board text added: "!LED_1"
- board text added: "!LED_2"
- board text added: "!LIGHT_INT"
- board text added: "!SD_CS"
- board text added: "0"
- board text added: "1"
- board text added: "2"
- board text added: "ACCEL_X"
- board text added: "ACCEL_Y"
- board text added: "ACCEL_Z"
- board text added: "GROVE_A0"
- board text added: "GROVE_A1"
- board text added: "GROVE_D0"
- board text added: "GROVE_D1"
- board text added: "LCD_MISO"
- board text added: "LCD_MOSI"
- board text added: "LCD_SCLK"
- board text added: "SD_EN"
- board text added: "SD_MISO"
- board text added: "SD_MOSI"
- board text added: "SD_SCLK"
- board text added: "TEMP & HUMIDITY"
- board text removed: "LED0"
- board text removed: "LED1"
- board text removed: "LED2"
- board text removed: "TEMPERATURE & HUMIDITY"

Commit message: Finished with revision B
Parts:
- removed R16: 100k, passives:0402_RES
- removed TP42: TEST_POINT_0.040IN, headers:TESTPOINT_0.040IN
- removed TP43, TP44: TEST_POINT_0.078IN, headers:TESTPOINT_0.078IN
- added R14: 100k, passives:0402_RES
- added TP21, TP30, TP32: TEST_POINT_0.040IN, headers:TESTPOINT_0.040IN
- J3, J4, J5: value 4P-2.0 -> (none)
- J6: value NRF52832DK_SHIELD -> (none); device headers:NRF52832DK_SHIELD -> headers:HW4-2.0
- J7: value 4P-2.0 -> NRF52832DK_SHIELD; device headers:HW4-2.0 -> headers:NRF52832DK_SHIELD
- TP40, TP41: value TEST_POINT_0.040IN -> TEST_POINT_0.078IN; device headers:TESTPOINT_0.040IN -> headers:TESTPOINT_0.078IN
- moved TP35 93.8 mm to (61.6, 0.00)
- moved J6 73.5 mm to (30.5, 10.2), turned to 90 degrees
- moved J7 73.5 mm to (7.62, 80.0), turned to 0 degrees
- moved TP36 69.8 mm to (1.91, 0.00)
- moved TP11 63.9 mm to (1.91, 47.0)
- moved TP26 63.9 mm to (1.91, 52.1)
- moved TP8 62.7 mm to (1.91, 54.6)
- moved TP41 61.6 mm to (2.54, 61.6)
- moved TP13 60.2 mm to (61.6, 54.6)
- moved TP28 60.1 mm to (1.91, 80.0)
- moved TP34 59.8 mm to (61.6, 81.5)
- moved TP31 59.7 mm to (1.91, 69.8)
- moved TP14 59.7 mm to (61.6, 44.5)
- moved TP39 57.4 mm to (61.6, 24.1)
- moved TP25 52.3 mm to (61.6, 86.6)
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- renumbered S5 to S4
Connections:
- net !BUTTON_0: now also J7.P0.28, TP26.TESTPOINT; no longer J6.P0.28, TP29.TESTPOINT
- net !IMU_INTERRUPT: now also J7.P0.07; no longer J6.P0.07
- net !LCD_CS: now also J7.P0.18; no longer J6.P0.18
- net !LED_0: now also J7.P0.25, TP5.TESTPOINT; no longer J6.P0.25, TP6.TESTPOINT
- net !LED_1: now also J7.P0.24, TP6.TESTPOINT; no longer J6.P0.24, TP7.TESTPOINT
- net !LED_2: now also J7.P0.23, TP7.TESTPOINT; no longer J6.P0.23, TP8.TESTPOINT
- net !LIGHT_INTERRUPT: now also J7.P0.27; no longer J6.P0.27
- net !RESET: now also J7.P0.21, TP39.TESTPOINT; no longer J6.P0.21, TP11.TESTPOINT
- net !SD_CS: now also J7.P0.14; no longer J6.P0.14
- net !SD_DETECT: now also R14.1, TP38.TESTPOINT; no longer R15.1, TP5.TESTPOINT
- net +3V3: now also J6.3, J7.3.3V@0, J7.3.3V@1, J7.3.3V@2, R15.2, TP28.TESTPOINT, TP29.TESTPOINT, TP30.TESTPOINT; no longer J6.3.3V@0, J6.3.3V@1, J6.3.3V@2, J7.3, R16.2, TP33.TESTPOINT, TP34.TESTPOINT, TP35.TESTPOINT
- net +5V: now also J7.5V, TP31.TESTPOINT; no longer J6.5V, TP36.TESTPOINT
- net ANALOG_ACCEL_X: now also J7.P0.29, TP10.TESTPOINT; no longer J6.P0.29, TP12.TESTPOINT
- net ANALOG_ACCEL_Y: now also J7.P0.30, TP11.TESTPOINT; no longer J6.P0.30, TP13.TESTPOINT
- net ANALOG_ACCEL_Z: now also J7.P0.31, TP12.TESTPOINT; no longer J6.P0.31, TP14.TESTPOINT
- net GND: now also J6.4, J7.GND@0, J7.GND@1, J7.GND@2, TP32.TESTPOINT, TP33.TESTPOINT, TP34.TESTPOINT, TP35.TESTPOINT, TP36.TESTPOINT, TP40.1, TP41.1; no longer J6.GND@0, J6.GND@1, J6.GND@2, J7.4, TP38.TESTPOINT, TP39.TESTPOINT, TP40.TESTPOINT, TP41.TESTPOINT, TP42.TESTPOINT, TP43.1, TP44.1
- net GROVE_A0: now also J7.P0.04, TP8.TESTPOINT; no longer J6.P0.04, TP9.TESTPOINT
- net GROVE_A1: now also J7.P0.03, TP9.TESTPOINT; no longer J6.P0.03, TP10.TESTPOINT
- net GROVE_D0: now also J6.1, J7.P0.02, TP24.TESTPOINT; no longer J6.P0.02, J7.1, TP27.TESTPOINT
- net GROVE_D1: now also J6.2, J7.P0.05, TP19.TESTPOINT; no longer J6.P0.05, J7.2, TP22.TESTPOINT
- net LCD_MISO: now also J7.P0.16, TP15.TESTPOINT; no longer J6.P0.16, TP17.TESTPOINT
- net LCD_MOSI: now also J7.P0.15, TP13.TESTPOINT; no longer J6.P0.15, TP15.TESTPOINT
- net LCD_SCLK: now also J7.P0.17, TP17.TESTPOINT; no longer J6.P0.17, TP19.TESTPOINT
- net N$18: now also R14.2; no longer R15.2
- net SD_ENABLE: now also J7.P0.26, R15.1, TP25.TESTPOINT; no longer J6.P0.26, R16.1, TP28.TESTPOINT
- net SD_MISO: now also J7.P0.12, TP16.TESTPOINT; no longer J6.P0.12, TP18.TESTPOINT
- net SD_MOSI: now also J7.P0.11, TP14.TESTPOINT; no longer J6.P0.11, TP16.TESTPOINT
- net SD_SCLK: now also J7.P0.13, TP18.TESTPOINT; no longer J6.P0.13, TP20.TESTPOINT
- net SENSORS_SCL: now also J7.P0.19, TP20.TESTPOINT; no longer J6.P0.19, TP23.TESTPOINT
- net SENSORS_SDA: now also J7.P0.20, TP21.TESTPOINT; no longer J6.P0.20, TP24.TESTPOINT
- net SWITCH_0: now also J7.P0.22, TP27.TESTPOINT; no longer J6.P0.22, TP31.TESTPOINT
- net UART_RX: now also J7.P0.08, TP22.TESTPOINT; no longer J6.P0.08, TP25.TESTPOINT
- net UART_TX: now also J7.P0.06, TP23.TESTPOINT; no longer J6.P0.06, TP26.TESTPOINT
Other:
- board text added: "+X"
- board text added: "+Y"
- board text added: "+Z"
- board text added: "."
