File: hardware/rev_b/buckler.sch (EAGLE design)
At the start: 90 parts, among them J1 DB25_5747846, J2 DM3AT-SF-PEJM5, J3 4P-2.0, J4 4P-2.0, J5 4P-2.0, J6 NRF52832DK_SHIELD, J7 4P-2.0, U1 ADXL327, U2 MAX44009, U3 MPU-9250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

Commit message: Routing complete
Connections:
- net N$1 renamed !RESET
- net N$2 renamed 5V_IN
- removed net EXTERN_RX: J1.1, J4.2
- net GROVE_A0: now also J6.P0.04/AIN2; no longer J6.P0.03/AIN1
- net GROVE_A1: now also J6.P0.03/AIN1; no longer J6.P0.04/AIN2
- net UART_RX: now also J1.1, J4.2
Other:
- moved on the sheet: TP10, TP9
Changed lines of the file:
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@@
 <instance part="TP7" gate="G$1" x="45.72" y="132.08"/>
 <instance part="TP8" gate="G$1" x="45.72" y="134.62"/>
-<instance part="TP9" gate="G$1" x="111.76" y="152.4" rot="R180"/>
-<instance part="TP10" gate="G$1" x="111.76" y="149.86" rot="R180"/>
+<instance part="TP9" gate="G$1" x="111.76" y="149.86" rot="R180"/>
+<instance part="TP10" gate="G$1" x="111.76" y="152.4" rot="R180"/>
 <instance part="TP12" gate="G$1" x="45.72" y="119.38" rot="MR180"/>
 <instance part="TP13" gate="G$1" x="45.72" y="116.84" rot="MR180"/>
@@
 </segment>
 </net>
-<net name="EXTERN_RX" class="0">
-<segment>
-<pinref part="J1" gate="J1" pin="1"/>
-<wire x1="203.2" y1="139.7" x2="200.66" y2="139.7" width="0.1524" layer="91"/>
-<label x="200.66" y="139.7" size="1.27" layer="95" font="vector" rot="R180" xref="yes"/>
-</segment>
-<segment>
-<pinref part="J4" gate="G$1" pin="2"/>
-<wire x1="99.06" y1="60.96" x2="93.98" y2="60.96" width="0.1524" layer="91"/>
-<label x="93.98" y="60.96" size="1.27" layer="95" font="vector" rot="R180" xref="yes"/>
-</segment>
-</net>
-<net name="N$2" class="0">
+<net name="5V_IN" class="0">
 <segment>
 <pinref part="J1" gate="J1" pin="8"/>
@@
 </segment>
 </net>
-<net name="N$1" class="0">
+<net name="!RESET" class="0">
 <segment>
 <wire x1="38.1" y1="152.4" x2="48.26" y2="152.4" width="0.1524" layer="91"/>
@@
 <label x="38.1" y="137.16" size="1.27" layer="95" font="vector" rot="R180" xref="yes"/>
 <pinref part="TP31" gate="G$1" pin="TESTPOINT"/>
-<wire x1="48.26" y1="137.16" x2="45.72" y2="137.16" width="0.1524" layer="91"/>
+<wire x1="48.26" y1="137.16" x2="38.1" y2="137.16" width="0.1524" layer="91"/>
 <junction x="48.26" y="137.16"/>
 <pinref part="J6" gate="J1" pin="P0.22"/>
-<wire x1="45.72" y1="137.16" x2="38.1" y2="137.16" width="0.1524" layer="91"/>
-<wire x1="48.26" y1="137.16" x2="45.72" y2="137.16" width="0.1524" layer="91"/>
+<wire x1="48.26" y1="137.16" x2="38.1" y2="137.16" width="0.1524" layer="91"/>
 </segment>
 </net>
@@
 </segment>
 <segment>
+<wire x1="106.68" y1="149.86" x2="109.22" y2="149.86" width="0.1524" layer="91"/>
+<label x="119.38" y="149.86" size="1.27" layer="95" font="vector" xref="yes"/>
+<pinref part="TP9" gate="G$1" pin="TESTPOINT"/>
+<wire x1="109.22" y1="149.86" x2="119.38" y2="149.86" width="0.1524" layer="91"/>
+<junction x="109.22" y="149.86"/>
+<pinref part="J6" gate="J1" pin="P0.04/AIN2"/>
+</segment>
+</net>
+<net name="GROVE_A1" class="0">
+<segment>
+<pinref part="J5" gate="G$1" pin="2"/>
+<wire x1="99.06" y1="25.4" x2="93.98" y2="25.4" width="0.1524" layer="91"/>
+<label x="93.98" y="25.4" size="1.27" layer="95" font="vector" rot="R180" xref="yes"/>
+</segment>
+<segment>
 <wire x1="106.68" y1="152.4" x2="109.22" y2="152.4" width="0.1524" layer="91"/>
 <label x="119.38" y="152.4" size="1.27" layer="95" font="vector" xref="yes"/>
-<pinref part="TP9" gate="G$1" pin="TESTPOINT"/>
+<pinref part="TP10" gate="G$1" pin="TESTPOINT"/>
 <wire x1="109.22" y1="152.4" x2="119.38" y2="152.4" width="0.1524" layer="91"/>
 <junction x="109.22" y="152.4"/>
 <pinref part="J6" gate="J1" pin="P0.03/AIN1"/>
-</segment>
-</net>
-<net name="GROVE_A1" class="0">
-<segment>
-<pinref part="J5" gate="G$1" pin="2"/>
-<wire x1="99.06" y1="25.4" x2="93.98" y2="25.4" width="0.1524" layer="91"/>
-<label x="93.98" y="25.4" size="1.27" layer="95" font="vector" rot="R180" xref="yes"/>
-</segment>
-<segment>
-<wire x1="106.68" y1="149.86" x2="109.22" y2="149.86" width="0.1524" layer="91"/>
-<label x="119.38" y="149.86" size="1.27" layer="95" font="vector" xref="yes"/>
-<pinref part="TP10" gate="G$1" pin="TESTPOINT"/>
-<wire x1="109.22" y1="149.86" x2="119.38" y2="149.86" width="0.1524" layer="91"/>
-<junction x="109.22" y="149.86"/>
-<pinref part="J6" gate="J1" pin="P0.04/AIN2"/>
 </segment>
 </net>
@@
 <pinref part="J6" gate="J1" pin="P0.08"/>
 </segment>
-</net>
+<segment>
+<pinref part="J1" gate="J1" pin="1"/>
+<wire x1="203.2" y1="139.7" x2="200.66" y2="139.7" width="0.1524" layer="91"/>
+<label x="200.66" y="139.7" size="1.27" layer="95" font="vector" rot="R180" xref="yes"/>
+</segment>
+<segment>
+<pinref part="J4" gate="G$1" pin="2"/>
+<wire x1="99.06" y1="60.96" x2="93.98" y2="60.96" width="0.1524" layer="91"/>
+<label x="93.98" y="60.96" size="1.27" layer="95" font="vector" rot="R180" xref="yes"/>
+</segment>
+</net>

Commit message: Finished with revision B
Parts:
- removed R16: 100k, passives:RESISTOR0402_RES
- removed TP42: TEST_POINT_0.040IN, headers:TEST_POINT_0.040IN
- removed TP43, TP44: TEST_POINT_0.078IN, headers:TEST_POINT_0.078IN
- added R14: 100k, passives:RESISTOR0402_RES
- added TP21, TP30, TP32: TEST_POINT_0.040IN, headers:TEST_POINT_0.040IN
- A1: DIGIKEY3 (none) -> 952-1862-ND
- J3, J4, J5: value 4P-2.0 -> GROVE-CONNECTOR-DIP(4P-2.0)
- J6: value NRF52832DK_SHIELD -> GROVE-CONNECTOR-DIP(4P-2.0); device headers:NRF52832DK_SHIELD -> headers:GROVE-CONNECTOR-DIP(4P-2.0); DESCRIPTION (none) -> Grove - Universal 4 pin connector; MANUFACTURER (none) -> Seeed Studio; MOUSER (none) -> 713-110990030; MPN (none) -> 110990030
- J7: value 4P-2.0 -> NRF52832DK_SHIELD; device headers:GROVE-CONNECTOR-DIP(4P-2.0) -> headers:NRF52832DK_SHIELD; DESCRIPTION Grove - Universal 4 pin connector -> (none); DIGIKEY1 (none) -> S1011EC-10-ND; DIGIKEY2 (none) -> S1011EC-08-ND; DIGIKEY3 (none) -> S1011EC-08-ND; DIGIKEY4 (none) -> S1011EC-06-ND; DIGIKEY5 (none) -> S1011EC-09-ND; MANUFACTURER Seeed Studio -> (none); MOUSER 713-110990030 -> (none); MPN 110990030 -> (none)
- TP40, TP41: value TEST_POINT_0.040IN -> TEST_POINT_0.078IN; device headers:TEST_POINT_0.040IN -> headers:TEST_POINT_0.078IN; DESCRIPTION (none) -> TERM TURRET SINGLE L=4.75MM TIN; DIGIKEY (none) -> 36-1520-2-ND; MANUFACTURER (none) -> Keystone Electronics; MPN (none) -> 1520-2
- renumbered S5 to S4
Connections:
- net !BUTTON_0: now also J7.P0.28/AIN4, TP26.TESTPOINT; no longer J6.P0.28/AIN4, TP29.TESTPOINT
- net !IMU_INTERRUPT: now also J7.P0.07; no longer J6.P0.07
- net !LCD_CS: now also J7.P0.18; no longer J6.P0.18
- net !LED_0: now also J7.P0.25, TP5.TESTPOINT; no longer J6.P0.25, TP6.TESTPOINT
- net !LED_1: now also J7.P0.24, TP6.TESTPOINT; no longer J6.P0.24, TP7.TESTPOINT
- net !LED_2: now also J7.P0.23, TP7.TESTPOINT; no longer J6.P0.23, TP8.TESTPOINT
- net !LIGHT_INTERRUPT: now also J7.P0.27; no longer J6.P0.27
- net !RESET: now also J7.P0.21/RESET, TP39.TESTPOINT; no longer J6.P0.21/RESET, TP11.TESTPOINT
- net !SD_CS: now also J7.P0.14; no longer J6.P0.14
- net !SD_DETECT: now also R14.1, TP38.TESTPOINT; no longer R15.1, TP5.TESTPOINT
- net +3V3: now also J6.3, J7.3.3V, R15.2, TP28.TESTPOINT, TP29.TESTPOINT, TP30.TESTPOINT; no longer J6.3.3V, J7.3, R16.2, TP33.TESTPOINT, TP34.TESTPOINT, TP35.TESTPOINT
- net +5V: now also J7.5V, TP31.TESTPOINT; no longer J6.5V, TP36.TESTPOINT
- net ANALOG_ACCEL_X: now also J7.P0.29/AIN5, TP10.TESTPOINT; no longer J6.P0.29/AIN5, TP12.TESTPOINT
- net ANALOG_ACCEL_Y: now also J7.P0.30/AIN6, TP11.TESTPOINT; no longer J6.P0.30/AIN6, TP13.TESTPOINT
- net ANALOG_ACCEL_Z: now also J7.P0.31/AIN7, TP12.TESTPOINT; no longer J6.P0.31/AIN7, TP14.TESTPOINT
- net GND: now also J6.4, J7.GND, TP32.TESTPOINT, TP33.TESTPOINT, TP34.TESTPOINT, TP35.TESTPOINT, TP36.TESTPOINT; no longer J6.GND, J7.4, TP38.TESTPOINT, TP39.TESTPOINT, TP42.TESTPOINT, TP43.TESTPOINT, TP44.TESTPOINT
- net GROVE_A0: now also J7.P0.04/AIN2, TP8.TESTPOINT; no longer J6.P0.04/AIN2, TP9.TESTPOINT
- net GROVE_A1: now also J7.P0.03/AIN1, TP9.TESTPOINT; no longer J6.P0.03/AIN1, TP10.TESTPOINT
- net GROVE_D0: now also J6.1, J7.P0.02/AIN0, TP24.TESTPOINT; no longer J6.P0.02/AIN0, J7.1, TP27.TESTPOINT
- net GROVE_D1: now also J6.2, J7.P0.05/AIN3, TP19.TESTPOINT; no longer J6.P0.05/AIN3, J7.2, TP22.TESTPOINT
- net LCD_MISO: now also J7.P0.16, TP15.TESTPOINT; no longer J6.P0.16, TP17.TESTPOINT
- net LCD_MOSI: now also J7.P0.15, TP13.TESTPOINT; no longer J6.P0.15, TP15.TESTPOINT
- net LCD_SCLK: now also J7.P0.17, TP17.TESTPOINT; no longer J6.P0.17, TP19.TESTPOINT
- net N$18: now also R14.2; no longer R15.2
- net SD_ENABLE: now also J7.P0.26, R15.1, TP25.TESTPOINT; no longer J6.P0.26, R16.1, TP28.TESTPOINT
- net SD_MISO: now also J7.P0.12, TP16.TESTPOINT; no longer J6.P0.12, TP18.TESTPOINT
- net SD_MOSI: now also J7.P0.11, TP14.TESTPOINT; no longer J6.P0.11, TP16.TESTPOINT
- net SD_SCLK: now also J7.P0.13, TP18.TESTPOINT; no longer J6.P0.13, TP20.TESTPOINT
- net SENSORS_SCL: now also J7.P0.19, TP20.TESTPOINT; no longer J6.P0.19, TP23.TESTPOINT
- net SENSORS_SDA: now also J7.P0.20, TP21.TESTPOINT; no longer J6.P0.20, TP24.TESTPOINT
- net SWITCH_0: now also J7.P0.22, TP27.TESTPOINT; no longer J6.P0.22, TP31.TESTPOINT
- net UART_RX: now also J7.P0.08, TP22.TESTPOINT; no longer J6.P0.08, TP25.TESTPOINT
- net UART_TX: now also J7.P0.06, TP23.TESTPOINT; no longer J6.P0.06, TP26.TESTPOINT
Other:
- moved on the sheet: R15, TP10, TP11, TP12, TP13, TP14, TP15, TP16, TP17, TP18, TP19, TP20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
